File: one/one/dac.kicad_sch (KiCad schematic)
At the start: 4 parts, among them U401 LTC2534

Commit message: add EEPROM, remove one mounting hole
Other:
- company: (none) -> ${LINK}
Changed lines of the file:
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@@
 	(title_block
 		(title "${TITLE}")
-		(date "2025-01-04")
+		(date "2025-01-06")
 		(rev "${REVISION}")
+		(company "${LINK}")
+		(comment 1 "${AUTHOR}")
 	)
 	(junction

Commit message: add vendor links
Parts:
- C401: Digikey (none) -> https://www.digikey.de/en/products/detail/cal-chip-electron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; MPN (none) -> GMC10X7R104K50NT; Tolerance (none) -> 20%; Voltage (none) -> 6V
- C402: Digikey (none) -> https://www.digikey.de/en/products/detail/cal-chip-electron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; MPN (none) -> GMC10X5R106M10NT
- FB401: value FerriteBead -> BLM18KG121TN1D; Digikey (none) -> https://www.digikey.de/en/products/detail/murata-electronic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; MPN (none) -> BLM18KG121TN1D
Changed lines of the file:
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@@
 	(title_block
 		(title "${TITLE}")
-		(date "2025-01-06")
+		(date "2025-01-26")
 		(rev "${REVISION}")
 		(company "${LINK}")
@@
 			)
 		)
-		(property "Datasheet" "~"
+		(property "Datasheet" "https://calchip.com/wp-content/uploads/2023/09/GMC-Series-2.pdf"
 			(at 134.62 114.3 0)
 			(effects
@@
 			)
 		)
-		(property "Description" "Unpolarized capacitor, small symbol"
+		(property "Description" "10 µF ±20% 10V Ceramic Capacitor X5R 0603 (1608 Metric)"
 			(at 134.62 114.3 0)
 			(effects
@@
 			)
 		)
-		(property "MPN" ""
+		(property "MPN" "GMC10X5R106M10NT"
 			(at 134.62 114.3 0)
 			(effects
@@
 			)
 		)
-		(property "Digikey" ""
+		(property "Digikey" "https://www.digikey.de/en/products/detail/cal-chip-electronics-inc/GMC10X5R106M10NT/18151101"
 			(at 134.62 114.3 0)
 			(effects
@@
 			)
 		)
-		(property "Value" "FerriteBead"
+		(property "Value" "BLM18KG121TN1D"
 			(at 103.5558 62.23 90)
 			(effects
@@
 			)
 		)
-		(property "Datasheet" "~"
+		(property "Datasheet" "https://www.murata.com/products/productdata/8796738650142/ENFA0003.pdf"
 			(at 103.505 66.675 0)
 			(effects
@@
 			)
 		)
-		(property "Description" "Ferrite bead"
+		(property "Description" "120 Ohms @ 100 MHz 1 Power Line Ferrite Bead 0603 (1608 Metric) 3A 30mOhm"
 			(at 103.505 66.675 0)
 			(effects
@@
 			)
 		)
-		(property "MPN" ""
+		(property "MPN" "BLM18KG121TN1D"
 			(at 103.505 66.675 90)
 			(effects
@@
 			)
 		)
-		(property "Digikey" ""
+		(property "Digikey" "https://www.digikey.de/en/products/detail/murata-electronics/BLM18KG121TN1D/1982762"
 			(at 103.505 66.675 90)
 			(effects
@@
 			)
 		)
-		(property "Datasheet" "~"
+		(property "Datasheet" "https://calchip.com/wp-content/uploads/2023/09/GMC-Series-2.pdf"
 			(at 120.015 72.39 0)
 			(effects
@@
 			)
 		)
-		(property "Description" "Unpolarized capacitor, small symbol"
+		(property "Description" "0.1 µF ±10% 50V Ceramic Capacitor X7R 0603 (1608 Metric)"
 			(at 120.015 72.39 0)
 			(effects
@@
 			)
 		)
-		(property "MPN" ""
+		(property "MPN" "GMC10X7R104K50NT"
 			(at 120.015 72.39 0)
 			(effects
@@
 			)
 		)
-		(property "Digikey" ""
+		(property "Digikey" "https://www.digikey.de/en/products/detail/cal-chip-electronics-inc/GMC10X7R104K50NT/18151094"
 			(at 120.015 72.39 0)
 			(effects
@@
 			)
 		)
-		(property "Voltage" ""
+		(property "Voltage" "6V"
 			(at 120.015 72.39 0)
 			(effects
@@
 			)
 		)
-		(property "Tolerance" ""
+		(property "Tolerance" "20%"
 			(at 120.015 72.39 0)
 			(effects
