File: one/one/io.kicad_sch (KiCad schematic)
At the start: 12 parts, among them Q1001 CPH5504, U1001 MOCD217M, U1002 MOCD217M

Commit message: add footprints
Parts:
- Q1001: footprint rpi:TSOT-23-5-mirrored -> hats:TSOT-23-5-mirrored
Changed lines of the file:
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@@
 		(date "2025-01-04")
 		(rev "${REVISION}")
-		(comment 1 "${AUTHOR}")
 	)
 	(junction
@@
 			)
 		)
-		(property "Footprint" "rpi:TSOT-23-5-mirrored"
+		(property "Footprint" "hats:TSOT-23-5-mirrored"
 			(at 217.17 94.361 0)
 			(effects

Commit message: add EEPROM, remove one mounting hole
Other:
- company: (none) -> ${LINK}
Changed lines of the file:
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@@
 	(title_block
 		(title "${TITLE}")
-		(date "2025-01-04")
+		(date "2025-01-06")
 		(rev "${REVISION}")
+		(company "${LINK}")
+		(comment 1 "${AUTHOR}")
 	)
 	(junction
