File: one/one/mechanical.kicad_sch (KiCad schematic)
At the start: 4 parts

Commit message: add EEPROM, remove one mounting hole
Parts:
- removed H802: M3, Mounting_Wuerth:Mounting_Wuerth_WA-SMSI-M3_H1mm_9774010360, symbol Mechanical:MountingHole
- H801, H803, H804: footprint Mounting_Wuerth:Mounting_Wuerth_WA-SMSI-M3_H1mm_9774010360 -> MountingHole:MountingHole_3.2mm_M3_DIN965; MPN 9774010360 -> (none)
Other:
- company: (none) -> ${LINK}
Changed lines of the file:
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@@
 	(title_block
 		(title "${TITLE}")
-		(date "2025-01-04")
+		(date "2025-01-06")
 		(rev "${REVISION}")
+		(company "${LINK}")
+		(comment 1 "${AUTHOR}")
 	)
 	(symbol
@@
 			)
 		)
-		(property "Footprint" "Mounting_Wuerth:Mounting_Wuerth_WA-SMSI-M3_H1mm_9774010360"
+		(property "Footprint" "MountingHole:MountingHole_3.2mm_M3_DIN965"
 			(at 50.165 167.64 0)
 			(effects
@@
 			)
 		)
-		(property "MPN" "9774010360"
+		(property "MPN" ""
 			(at 50.165 167.64 0)
 			(effects
@@
 				(path "/ed16f909-220f-4714-ae8c-981e375876e1/6aeb8ee1-e5ac-4174-9f06-8edc9b25f36b"
 					(reference "H801")
-					(unit 1)
-				)
-			)
-		)
-	)
-	(symbol
-		(lib_id "Mechanical:MountingHole")
-		(at 50.165 177.8 0)
-		(unit 1)
-		(exclude_from_sim yes)
-		(in_bom no)
-		(on_board yes)
-		(dnp no)
-		(fields_autoplaced yes)
-		(property "Reference" "H802"
-			(at 52.705 176.5299 0)
-			(effects
-				(font
-					(size 1.27 1.27)
-				)
-				(justify left)
-			)
-		)
-		(property "Value" "M3"
-			(at 52.705 179.0699 0)
-			(effects
-				(font
-					(size 1.27 1.27)
-				)
-				(justify left)
-			)
-		)
-		(property "Footprint" "Mounting_Wuerth:Mounting_Wuerth_WA-SMSI-M3_H1mm_9774010360"
-			(at 50.165 177.8 0)
-			(effects
-				(font
-					(size 1.27 1.27)
-				)
-				(hide yes)
-			)
-		)
-		(property "Datasheet" "~"
-			(at 50.165 177.8 0)
-			(effects
-				(font
-					(size 1.27 1.27)
-				)
-				(hide yes)
-			)
-		)
-		(property "Description" "Mounting Hole without connection"
-			(at 50.165 177.8 0)
-			(effects
-				(font
-					(size 1.27 1.27)
-				)
-				(hide yes)
-			)
-		)
-		(property "MPN" "9774010360"
-			(at 50.165 177.8 0)
-			(effects
-				(font
-					(size 1.27 1.27)
-				)
-				(hide yes)
-			)
-		)
-		(property "Digikey" ""
-			(at 50.165 177.8 0)
-			(effects
-				(font
-					(size 1.27 1.27)
-				)
-				(hide yes)
-			)
-		)
-		(property "Mouser" ""
-			(at 50.165 177.8 0)
-			(effects
-				(font
-					(size 1.27 1.27)
-				)
-				(hide yes)
-			)
-		)
-		(property "Price" ""
-			(at 50.165 177.8 0)
-			(effects
-				(font
-					(size 1.27 1.27)
-				)
-				(hide yes)
-			)
-		)
-		(instances
-			(project "rpi"
-				(path "/ed16f909-220f-4714-ae8c-981e375876e1/6aeb8ee1-e5ac-4174-9f06-8edc9b25f36b"
-					(reference "H802")
 					(unit 1)
 				)
@@
 			)
 		)
-		(property "Footprint" "Mounting_Wuerth:Mounting_Wuerth_WA-SMSI-M3_H1mm_9774010360"
+		(property "Footprint" "MountingHole:MountingHole_3.2mm_M3_DIN965"
 			(at 67.31 168.275 0)
 			(effects
@@
 			)
 		)
-		(property "MPN" "9774010360"
+		(property "MPN" ""
 			(at 67.31 168.275 0)
 			(effects
@@
 			)
 		)
-		(property "Footprint" "Mounting_Wuerth:Mounting_Wuerth_WA-SMSI-M3_H1mm_9774010360"
+		(property "Footprint" "MountingHole:MountingHole_3.2mm_M3_DIN965"
 			(at 67.31 177.165 0)
 			(effects
@@
 			)
 		)
-		(property "MPN" "9774010360"
-			(at 67.31 177.165 0)
-			(effects
+		(property "MPN" ""
+			(at 67.31 177.165 0)
+			(effects
