File: one/one/one.kicad_sch (KiCad schematic)
At the start: 14 parts, among them J101 Conn_01x04_Pin, J102 Conn_01x04_Pin, J103 ADC, J104 DAC, J105 SJ-252X, J106 Conn_01x04_Pin, J107 Conn_01x04_Pin, J108 Conn_02x04_Counter_Clockwise, J109 Conn_01x04_Pin, J110 Conn_01x05_Pin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

Commit message: add footprints
Parts:
- J105, J113: footprint rpi:SJ-252X -> hats:SJ-252X; Digikey (none) -> https://www.digikey.de/product-detail/de/cui-inc/SJ-2523-SM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; Price (none) -> 0.85; Price (EUR) 0.85 -> (none); Price100 (EUR) 0.65 -> (none); Source1 https://www.digikey.de/product-detail/de/cui-inc/SJ-2523-SM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 -> (none)
- J111: footprint rpi:SJ-3524 -> hatsi:SJ-3524; Digikey (none) -> https://www.digikey.de/product-detail/de/cui-inc/SJ-3524-SM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; Price (none) -> 1.07; Price (EUR) 1.07 -> (none); Price100 (EUR) 0.81 -> (none); Source1 https://www.digikey.de/product-detail/de/cui-inc/SJ-3524-SM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 -> (none)
Other:
- company: (none) -> ${LINK}
Changed lines of the file:
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@@
 		(date "2025-01-04")
 		(rev "${REVISION}")
+		(company "${LINK}")
 		(comment 1 "${AUTHOR}")
 	)
@@
 			)
 		)
-		(property "Footprint" "rpi:SJ-252X"
+		(property "Footprint" "hats:SJ-252X"
 			(at 163.83 115.57 0)
 			(effects
@@
 			)
 		)
-		(property "Source1" "https://www.digikey.de/product-detail/de/cui-inc/SJ-2523-SMT-TR/CP-2523SJCT-ND/669702"
-			(at 163.83 106.045 0)
-			(effects
-				(font
-					(size 1.524 1.524)
-				)
-				(hide yes)
-			)
-		)
-		(property "Source2" "~"
-			(at 163.83 106.045 0)
-			(effects
-				(font
-					(size 1.524 1.524)
-				)
-				(hide yes)
-			)
-		)
-		(property "Comment" "~"
+		(property "MPN" "SJ-2523-SMT-TR"
 			(at 163.83 106.045 0)
 			(effects
@@
 			)
 		)
-		(property "Critical" "~"
+		(property "Digikey" "https://www.digikey.de/product-detail/de/cui-inc/SJ-2523-SMT-TR/CP-2523SJCT-ND/669702"
 			(at 163.83 106.045 0)
 			(effects
@@
 			)
 		)
-		(property "MPN" "SJ-2523-SMT-TR"
+		(property "Mouser" "~"
 			(at 163.83 106.045 0)
 			(effects
@@
 			)
 		)
-		(property "Price (EUR)" "0.85"
-			(at 163.83 106.045 0)
-			(effects
-				(font
-					(size 1.27 1.27)
-				)
-				(hide yes)
-			)
-		)
-		(property "Price100 (EUR)" "0.65"
+		(property "Price" "0.85"
 			(at 163.83 106.045 0)
 			(effects
@@
 			)
 		)
-		(property "Footprint" "rpi:SJ-252X"
+		(property "Footprint" "hats:SJ-252X"
 			(at 163.83 102.235 0)
 			(effects
@@
 			)
 		)
-		(property "Source1" "https://www.digikey.de/product-detail/de/cui-inc/SJ-2523-SMT-TR/CP-2523SJCT-ND/669702"
-			(at 163.83 92.71 0)
-			(effects
-				(font
-					(size 1.524 1.524)
-				)
-				(hide yes)
-			)
-		)
-		(property "Source2" "~"
-			(at 163.83 92.71 0)
-			(effects
-				(font
-					(size 1.524 1.524)
-				)
-				(hide yes)
-			)
-		)
-		(property "Comment" "~"
+		(property "MPN" "SJ-2523-SMT-TR"
 			(at 163.83 92.71 0)
 			(effects
@@
 			)
 		)
-		(property "Critical" "~"
+		(property "Digikey" "https://www.digikey.de/product-detail/de/cui-inc/SJ-2523-SMT-TR/CP-2523SJCT-ND/669702"
 			(at 163.83 92.71 0)
 			(effects
@@
 			)
 		)
-		(property "MPN" "SJ-2523-SMT-TR"
+		(property "Mouser" "~"
 			(at 163.83 92.71 0)
 			(effects
@@
 			)
 		)
-		(property "Price (EUR)" "0.85"
-			(at 163.83 92.71 0)
-			(effects
-				(font
-					(size 1.27 1.27)
-				)
-				(hide yes)
-			)
-		)
-		(property "Price100 (EUR)" "0.65"
+		(property "Price" "0.85"
 			(at 163.83 92.71 0)
 			(effects
@@
 			)
 		)
-		(property "Footprint" "rpi:SJ-3524"
+		(property "Footprint" "hatsi:SJ-3524"
 			(at 163.83 111.76 0)
 			(effects
@@
 			)
 		)
-		(property "Source1" "https://www.digikey.de/product-detail/de/cui-inc/SJ-3524-SMT-TR-PI/CP-3524SJPICT-ND/2296006"
-			(at 163.83 121.285 0)
-			(effects
-				(font
-					(size 1.524 1.524)
-				)
-				(hide yes)
-			)
-		)
-		(property "Source2" "~"
+		(property "MPN" "SJ-3524-SMT-TR-PI"
 			(at 163.83 121.285 0)
 			(effects
@@
 			)
 		)
-		(property "Comment" "~"
+		(property "Digikey" "https://www.digikey.de/product-detail/de/cui-inc/SJ-3524-SMT-TR-PI/CP-3524SJPICT-ND/2296006"
 			(at 163.83 121.285 0)
 			(effects
@@
 			)
 		)
-		(property "Critical" "~"
+		(property "Mouser" "~"
 			(at 163.83 121.285 0)
 			(effects
@@
 			)
 		)
-		(property "MPN" "SJ-3524-SMT-TR-PI"
-			(at 163.83 121.285 0)
-			(effects
-				(font
-					(size 1.524 1.524)
-				)
-				(hide yes)
-			)
-		)
-		(property "Price (EUR)" "1.07"
-			(at 163.83 121.285 0)
-			(effects
-				(font
-					(size 1.27 1.27)
-				)
-				(hide yes)
-			)
-		)
-		(property "Price100 (EUR)" "0.81"
+		(property "Price" "1.07"
 			(at 163.83 121.285 0)
 			(effects
@@
 		)
 		(instances
-			(project "analogue"
+			(project "one"
 				(path "/ed16f909-220f-4714-ae8c-981e375876e1"
 					(page "9")
@@
 		)
 		(instances
-			(project "analogue"
+			(project "one"
 				(path "/ed16f909-220f-4714-ae8c-981e375876e1"
 					(page "3")
@@
 		)
 		(instances
-			(project "analogue"
+			(project "one"
 				(path "/ed16f909-220f-4714-ae8c-981e375876e1"
 					(page "8")
@@
 		)
 		(instances
-			(project "analogue"
+			(project "one"
 				(path "/ed16f909-220f-4714-ae8c-981e375876e1"
 					(page "7")
@@
 		)
 		(instances
-			(project "analogue"
+			(project "one"
 				(path "/ed16f909-220f-4714-ae8c-981e375876e1"
 					(page "6")
@@
 		)
 		(instances
-			(project "analogue"
+			(project "one"
 				(path "/ed16f909-220f-4714-ae8c-981e375876e1"
 					(page "10")
@@
 		)
 		(instances
-			(project "analogue"
+			(project "one"
 				(path "/ed16f909-220f-4714-ae8c-981e375876e1"
 					(page "4")
@@
 		)
 		(instances
-			(project "analogue"
+			(project "one"
 				(path "/ed16f909-220f-4714-ae8c-981e375876e1"
 					(page "2")
@@
 		)
 		(instances
-			(project "analogue"
+			(project "one"
 				(path "/ed16f909-220f-4714-ae8c-981e375876e1"
 					(page "5")

Commit message: add vendor links
Parts:
- C101: Digikey (none) -> https://www.digikey.de/en/products/detail/cal-chip-electron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; MPN (none) -> GMC10X7R104K50NT
Changed lines of the file:
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@@
 	(title_block
 		(title "${TITLE}")
-		(date "2025-01-06")
+		(date "2025-01-26")
 		(rev "${REVISION}")
 		(company "${LINK}")
@@
 			)
 		)
-		(property "Datasheet" "~"
+		(property "Datasheet" "https://calchip.com/wp-content/uploads/2023/09/GMC-Series-2.pdf"
 			(at 263.525 45.085 0)
 			(effects
@@
 			)
 		)
-		(property "Description" "Unpolarized capacitor, small symbol"
+		(property "Description" "0.1 µF ±10% 50V Ceramic Capacitor X7R 0603 (1608 Metric)"
 			(at 263.525 45.085 0)
 			(effects
@@
 			)
 		)
-		(property "MPN" ""
+		(property "MPN" "GMC10X7R104K50NT"
 			(at 263.525 45.085 0)
 			(effects
@@
 			)
 		)
-		(property "Digikey" ""
+		(property "Digikey" "https://www.digikey.de/en/products/detail/cal-chip-electronics-inc/GMC10X7R104K50NT/18151094"
 			(at 263.525 45.085 0)
 			(effects
