File: one/one/power.kicad_sch (KiCad schematic)
At the start: 4 parts, among them J501 12V

Commit message: add footprints
Parts:
- J501: footprint rpi:CUI-PJ-018 -> hats:CUI-PJ-018; Digikey (none) -> https://www.digikey.de/de/products/detail/cui-devices/PJ-01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; Label V_{in} -> V_{in}<12V; Price (none) -> 0.58; Price (EUR) 0.58 -> (none); Price100 (EUR) 0.42 -> (none); Source1 https://www.digikey.de/de/products/detail/cui-devices/PJ-01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 -> (none)
Changed lines of the file:
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@@
 		(date "2025-01-04")
 		(rev "${REVISION}")
-		(comment 1 "${AUTHOR}")
 	)
 	(junction
@@
 			)
 		)
-		(property "Footprint" "rpi:CUI-PJ-018"
+		(property "Footprint" "hats:CUI-PJ-018"
 			(at 95.25 86.36 0)
 			(effects
@@
 			)
 		)
-		(property "Source1" "https://www.digikey.de/de/products/detail/cui-devices/PJ-018/1644612"
-			(at 94.615 94.615 0)
-			(effects
-				(font
-					(size 1.524 1.524)
-				)
-				(hide yes)
-			)
-		)
-		(property "Source2" "~"
-			(at 94.615 94.615 0)
-			(effects
-				(font
-					(size 1.524 1.524)
-				)
-				(hide yes)
-			)
-		)
-		(property "Comment" "~"
-			(at 94.615 94.615 0)
-			(effects
-				(font
-					(size 1.524 1.524)
-				)
-				(hide yes)
-			)
-		)
-		(property "Critical" "~"
-			(at 94.615 94.615 0)
-			(effects
-				(font
-					(size 1.524 1.524)
-				)
-				(hide yes)
-			)
-		)
 		(property "MPN" "PJ-018"
 			(at 94.615 94.615 0)
@@
 			)
 		)
-		(property "Price (EUR)" "0.58"
+		(property "Digikey" "https://www.digikey.de/de/products/detail/cui-devices/PJ-018/1644612"
 			(at 94.615 94.615 0)
 			(effects
 				(font
-					(size 1.27 1.27)
-				)
-				(hide yes)
-			)
-		)
-		(property "Price100 (EUR)" "0.42"
+					(size 1.524 1.524)
+				)
+				(hide yes)
+			)
+		)
+		(property "Mouser" "~"
 			(at 94.615 94.615 0)
 			(effects
 				(font
-					(size 1.27 1.27)
-				)
-				(hide yes)
-			)
-		)
-		(property "Label" "V_{in}"
+					(size 1.524 1.524)
+				)
+				(hide yes)
+			)
+		)
+		(property "Price" "0.58"
+			(at 94.615 94.615 0)
+			(effects
+				(font
+					(size 1.27 1.27)
+				)
+				(hide yes)
+			)
+		)
+		(property "Label" "V_{in}<12V"
 			(at 94.742 85.852 0)
 			(show_name yes)

Commit message: add EEPROM, remove one mounting hole
Other:
- company: (none) -> ${LINK}
Changed lines of the file:
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@@
 	(title_block
 		(title "${TITLE}")
-		(date "2025-01-04")
+		(date "2025-01-06")
 		(rev "${REVISION}")
+		(company "${LINK}")
+		(comment 1 "${AUTHOR}")
 	)
 	(junction

Commit message: add vendor links
Parts:
- C501: Digikey (none) -> https://www.digikey.de/en/products/detail/cal-chip-electron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; MPN (none) -> GMC10X5R106M10NT; Tolerance (none) -> 20%; Voltage (none) -> 6
- C502: Digikey (none) -> https://www.digikey.de/en/products/detail/cal-chip-electron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; MPN (none) -> GMC10X7R104K50NT
- C503: Digikey (none) -> https://www.digikey.de/en/products/detail/chemi-con/APXG160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; MPN (none) -> APXG160ARA101ME61G; Price (none) -> 0.6; Tolerance (none) -> 20%; Voltage (none) -> 16V
Other:
- moved on the sheet: C503
Changed lines of the file:
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@@
 	(title_block
 		(title "${TITLE}")
-		(date "2025-01-06")
+		(date "2025-01-26")
 		(rev "${REVISION}")
 		(company "${LINK}")
@@
 	(wire
 		(pts
-			(xy 143.51 93.98) (xy 143.51 90.17)
+			(xy 143.51 92.71) (xy 143.51 90.17)
 		)
 		(stroke
@@
 	(wire
 		(pts
-			(xy 143.51 99.06) (xy 143.51 100.33)
+			(xy 143.51 97.79) (xy 143.51 100.33)
 		)
 		(stroke
@@
 		(shape output)
 		(at 238.125 139.065 0)
-		(fields_autoplaced yes)
 		(effects
 			(font
@@
 		(shape output)
 		(at 238.125 135.255 0)
-		(fields_autoplaced yes)
 		(effects
 			(font
@@
 		(shape output)
 		(at 238.125 142.875 0)
-		(fields_autoplaced yes)
 		(effects
 			(font
@@
 			)
 		)
-		(property "Datasheet" "~"
+		(property "Datasheet" "https://calchip.com/wp-content/uploads/2023/09/GMC-Series-2.pdf"
 			(at 169.545 95.25 0)
 			(effects
@@
 			)
 		)
-		(property "Description" "Unpolarized capacitor, small symbol"
+		(property "Description" "0.1 µF ±10% 50V Ceramic Capacitor X7R 0603 (1608 Metric)"
 			(at 169.545 95.25 0)
 			(effects
@@
 			)
 		)
-		(property "MPN" ""
+		(property "MPN" "GMC10X7R104K50NT"
 			(at 169.545 95.25 0)
 			(effects
@@
 			)
 		)
-		(property "Digikey" ""
+		(property "Digikey" "https://www.digikey.de/en/products/detail/cal-chip-electronics-inc/GMC10X7R104K50NT/18151094"
 			(at 169.545 95.25 0)
 			(effects
@@
 	(symbol
 		(lib_id "Device:C_Polarized_Small")
-		(at 143.51 96.52 0)
+		(at 143.51 95.25 0)
 		(unit 1)
 		(exclude_from_sim no)
@@
 		(fields_autoplaced yes)
 		(property "Reference" "C503"
-			(at 146.685 94.7038 0)
+			(at 146.685 93.4338 0)
 			(effects
 				(font
@@
 		)
 		(property "Value" "100uF"
-			(at 146.685 97.2438 0)
+			(at 146.685 95.9738 0)
 			(effects
 				(font
@@
 		)
 		(property "Footprint" "Capacitor_SMD:C_Elec_5x5.8"
-			(at 143.51 96.52 0)
-			(effects
-				(font
-					(size 1.27 1.27)
-				)
-				(hide yes)
-			)
-		)
-		(property "Datasheet" "~"
-			(at 143.51 96.52 0)
-			(effects
-				(font
-					(size 1.27 1.27)
-				)
-				(hide yes)
-			)
-		)
-		(property "Description" "Polarized capacitor, small symbol"
-			(at 143.51 96.52 0)
-			(effects
-				(font
-					(size 1.27 1.27)
-				)
-				(hide yes)
-			)
-		)
-		(property "MPN" ""
-			(at 143.51 96.52 0)
-			(effects
-				(font
-					(size 1.27 1.27)
-				)
-				(hide yes)
-			)
-		)
-		(property "Digikey" ""
-			(at 143.51 96.52 0)
+			(at 143.51 95.25 0)
+			(effects
+				(font
+					(size 1.27 1.27)
+				)
+				(hide yes)
+			)
+		)
+		(property "Datasheet" "https://www.chemi-con.co.jp/products/relatedfiles/capacitor/catalog/PXGRA-e.PDF"
+			(at 143.51 95.25 0)
+			(effects
+				(font
+					(size 1.27 1.27)
+				)
+				(hide yes)
+			)
+		)
+		(property "Description" "100 µF 16 V Aluminum - Polymer Capacitors Radial, Can - SMD 27mOhm 15000 Hrs @ 105°C"
+			(at 143.51 95.25 0)
+			(effects
+				(font
+					(size 1.27 1.27)
+				)
+				(hide yes)
+			)
+		)
+		(property "MPN" "APXG160ARA101ME61G"
+			(at 143.51 95.25 0)
+			(effects
+				(font
+					(size 1.27 1.27)
+				)
+				(hide yes)
+			)
+		)
+		(property "Digikey" "https://www.digikey.de/en/products/detail/chemi-con/APXG160ARA101ME61G/3983370"
+			(at 143.51 95.25 0)
 			(effects
 				(font
@@
 		)
 		(property "Mouser" ""
-			(at 143.51 96.52 0)
-			(effects
-				(font
-					(size 1.27 1.27)
-				)
-				(hide yes)
-			)
-		)
-		(property "Voltage" ""
-			(at 143.51 96.52 0)
-			(effects
-				(font
-					(size 1.27 1.27)
-				)
-				(hide yes)
-			)
-		)
-		(property "Tolerance" ""
-			(at 143.51 96.52 0)
-			(effects
-				(font
-					(size 1.27 1.27)
-				)
-				(hide yes)
-			)
-		)
-		(property "Price" ""
-			(at 143.51 96.52 0)
+			(at 143.51 95.25 0)
+			(effects
+				(font
+					(size 1.27 1.27)
+				)
+				(hide yes)
+			)
+		)
+		(property "Voltage" "16V"
+			(at 143.51 95.25 0)
+			(effects
+				(font
+					(size 1.27 1.27)
+				)
+				(hide yes)
+			)
+		)
+		(property "Tolerance" "20%"
+			(at 143.51 95.25 0)
+			(effects
+				(font
+					(size 1.27 1.27)
+				)
+				(hide yes)
+			)
+		)
+		(property "Price" "0.6"
+			(at 143.51 95.25 0)
 			(effects
 				(font
@@
 			)
 		)
-		(property "Datasheet" "~"
+		(property "Datasheet" "https://calchip.com/wp-content/uploads/2023/09/GMC-Series-2.pdf"
 			(at 156.845 95.25 0)
 			(effects
@@
 			)
 		)
-		(property "Description" "Unpolarized capacitor, small symbol"
+		(property "Description" "10 µF ±20% 10V Ceramic Capacitor X5R 0603 (1608 Metric)"
 			(at 156.845 95.25 0)
 			(effects
@@
 			)
 		)
-		(property "MPN" ""
+		(property "MPN" "GMC10X5R106M10NT"
 			(at 156.845 95.25 0)
 			(effects
@@
 			)
 		)
-		(property "Digikey" ""
+		(property "Digikey" "https://www.digikey.de/en/products/detail/cal-chip-electronics-inc/GMC10X5R106M10NT/18151101"
 			(at 156.845 95.25 0)
 			(effects
@@
 			)
 		)
-		(property "Voltage" ""
+		(property "Voltage" "6"
 			(at 156.845 95.25 0)
 			(effects
@@
 			)
 		)
-		(property "Tolerance" ""
+		(property "Tolerance" "20%"
 			(at 156.845 95.25 0)
 			(effects
