File: one/one/rpi-interface.kicad_sch (KiCad schematic)
At the start: 3 parts, among them J201 Conn_02x20_Odd_Even

Commit message: add EEPROM, remove one mounting hole
Other:
- company: (none) -> ${LINK}
Changed lines of the file:
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@@
 	(title_block
 		(title "${TITLE}")
-		(date "2025-01-04")
+		(date "2025-01-06")
 		(rev "${REVISION}")
+		(company "${LINK}")
+		(comment 1 "${AUTHOR}")
 	)
 	(junction

Commit message: add vendor links
Parts:
- J201: value Conn_02x20_Odd_Even -> NPTC202KFMS-RC; Digikey (none) -> https://www.digikey.de/en/products/detail/sullins-connector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; MPN (none) -> NPTC202KFMS-RC; Price (none) -> 3.2
Changed lines of the file:
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@@
 	(title_block
 		(title "${TITLE}")
-		(date "2025-01-06")
+		(date "2025-01-26")
 		(rev "${REVISION}")
 		(company "${LINK}")
@@
 			)
 		)
-		(property "Value" "Conn_02x20_Odd_Even"
+		(property "Value" "NPTC202KFMS-RC"
 			(at 129.54 66.675 0)
 			(effects
@@
 			)
 		)
-		(property "Datasheet" "~"
+		(property "Datasheet" "https://mm.digikey.com/Volume0/opasdata/d220001/medias/docus/937/Female_Headers.100_DS.pdf"
 			(at 128.27 93.345 0)
 			(effects
@@
 			)
 		)
-		(property "Description" "Generic connector, double row, 02x20, odd/even pin numbering scheme (row 1 odd numbers, row 2 even numbers), script generated (kicad-library-utils/schlib/autogen/connector/)"
+		(property "Description" "40 Position Header Connector 0.100\" (2.54mm) Surface Mount Tin"
 			(at 128.27 93.345 0)
 			(effects
@@
 			)
 		)
-		(property "MPN" ""
+		(property "MPN" "NPTC202KFMS-RC"
+			(at 128.27 93.345 0)
+			(effects
+				(font
+					(size 1.27 1.27)
+				)
+				(hide yes)
+			)
+		)
+		(property "Digikey" "https://www.digikey.de/en/products/detail/sullins-connector-solutions/nptc202kfms-rc/776149"
 			(at 128.27 93.345 0)
 			(effects
@@
 			)
 		)
-		(property "Price" ""
+		(property "Price" "3.2"
 			(at 128.27 93.345 0)
 			(effects
