File: one/one/stepper-motor.kicad_sch (KiCad schematic)
At the start: 7 parts

Commit message: add EEPROM, remove one mounting hole
Other:
- company: (none) -> ${LINK}
Changed lines of the file:
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@@
 	(title_block
 		(title "${TITLE}")
-		(date "2025-01-04")
+		(date "2025-01-06")
 		(rev "${REVISION}")
+		(company "${LINK}")
+		(comment 1 "${AUTHOR}")
 	)
 	(junction

Commit message: add vendor links
Parts:
- C901, C904: Digikey (none) -> https://www.digikey.de/en/products/detail/cal-chip-electron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; MPN (none) -> GMC10X5R106M10NT
- C902, C905: Digikey (none) -> https://www.digikey.de/en/products/detail/cal-chip-electron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; MPN (none) -> GMC10X7R104K50NT
- C903: Digikey (none) -> https://www.digikey.de/en/products/detail/chemi-con/APXG160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; MPN (none) -> APXG160ARA101ME61G; Price (none) -> 0.6
- FB901: value FerriteBead -> BLM18KG121TN1D; Digikey (none) -> https://www.digikey.de/en/products/detail/murata-electronic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; MPN (none) -> BLM18KG121TN1D
Changed lines of the file:
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@@
 	(title_block
 		(title "${TITLE}")
-		(date "2025-01-06")
+		(date "2025-01-26")
 		(rev "${REVISION}")
 		(company "${LINK}")
@@
 		(shape output)
 		(at 155.575 109.22 0)
-		(fields_autoplaced yes)
 		(effects
 			(font
@@
 		(shape output)
 		(at 155.575 114.3 0)
-		(fields_autoplaced yes)
 		(effects
 			(font
@@
 		(shape output)
 		(at 155.575 106.68 0)
-		(fields_autoplaced yes)
 		(effects
 			(font
@@
 		(shape output)
 		(at 155.575 111.76 0)
-		(fields_autoplaced yes)
 		(effects
 			(font
@@
 			)
 		)
-		(property "Datasheet" "~"
+		(property "Datasheet" "https://www.chemi-con.co.jp/products/relatedfiles/capacitor/catalog/PXGRA-e.PDF"
 			(at 205.105 71.755 0)
 			(effects
@@
 			)
 		)
-		(property "Description" "Polarized capacitor, small symbol"
+		(property "Description" "100 µF 16 V Aluminum - Polymer Capacitors Radial, Can - SMD 27mOhm 15000 Hrs @ 105°C"
 			(at 205.105 71.755 0)
 			(effects
@@
 			)
 		)
-		(property "MPN" ""
+		(property "MPN" "APXG160ARA101ME61G"
 			(at 205.105 71.755 0)
 			(effects
@@
 			)
 		)
-		(property "Digikey" ""
+		(property "Digikey" "https://www.digikey.de/en/products/detail/chemi-con/APXG160ARA101ME61G/3983370"
 			(at 205.105 71.755 0)
 			(effects
@@
 			)
 		)
-		(property "Price" ""
+		(property "Price" "0.6"
 			(at 205.105 71.755 0)
 			(effects
@@
 			)
 		)
-		(property "Value" "FerriteBead"
+		(property "Value" "BLM18KG121TN1D"
 			(at 91.4908 58.42 90)
 			(effects
@@
 			)
 		)
-		(property "Datasheet" "~"
+		(property "Datasheet" "https://www.murata.com/products/productdata/8796738650142/ENFA0003.pdf"
 			(at 91.44 62.865 0)
 			(effects
@@
 			)
 		)
-		(property "Description" "Ferrite bead"
+		(property "Description" "120 Ohms @ 100 MHz 1 Power Line Ferrite Bead 0603 (1608 Metric) 3A 30mOhm"
 			(at 91.44 62.865 0)
 			(effects
@@
 			)
 		)
-		(property "MPN" ""
+		(property "MPN" "BLM18KG121TN1D"
 			(at 91.44 62.865 90)
 			(effects
@@
 			)
 		)
-		(property "Digikey" ""
+		(property "Digikey" "https://www.digikey.de/en/products/detail/murata-electronics/BLM18KG121TN1D/1982762"
 			(at 91.44 62.865 90)
 			(effects
@@
 			)
 		)
-		(property "Datasheet" "~"
+		(property "Datasheet" "https://calchip.com/wp-content/uploads/2023/09/GMC-Series-2.pdf"
 			(at 99.06 71.755 0)
 			(effects
@@
 			)
 		)
-		(property "Description" "Unpolarized capacitor, small symbol"
+		(property "Description" "10 µF ±20% 10V Ceramic Capacitor X5R 0603 (1608 Metric)"
 			(at 99.06 71.755 0)
 			(effects
@@
 			)
 		)
-		(property "MPN" ""
+		(property "MPN" "GMC10X5R106M10NT"
 			(at 99.06 71.755 0)
 			(effects
@@
 			)
 		)
-		(property "Digikey" ""
+		(property "Digikey" "https://www.digikey.de/en/products/detail/cal-chip-electronics-inc/GMC10X5R106M10NT/18151101"
 			(at 99.06 71.755 0)
 			(effects
@@
 			)
 		)
-		(property "Datasheet" "~"
+		(property "Datasheet" "https://calchip.com/wp-content/uploads/2023/09/GMC-Series-2.pdf"
 			(at 193.04 71.755 0)
 			(effects
@@
 			)
 		)
-		(property "Description" "Unpolarized capacitor, small symbol"
+		(property "Description" "10 µF ±20% 10V Ceramic Capacitor X5R 0603 (1608 Metric)"
 			(at 193.04 71.755 0)
 			(effects
@@
 			)
 		)
-		(property "MPN" ""
+		(property "MPN" "GMC10X5R106M10NT"
 			(at 193.04 71.755 0)
 			(effects
@@
 			)
 		)
-		(property "Digikey" ""
+		(property "Digikey" "https://www.digikey.de/en/products/detail/cal-chip-electronics-inc/GMC10X5R106M10NT/18151101"
 			(at 193.04 71.755 0)
 			(effects
@@
 			)
 		)
-		(property "Datasheet" "~"
+		(property "Datasheet" "https://calchip.com/wp-content/uploads/2023/09/GMC-Series-2.pdf"
 			(at 180.975 71.755 0)
 			(effects
@@
 			)
 		)
-		(property "Description" "Unpolarized capacitor, small symbol"
+		(property "Description" "0.1 µF ±10% 50V Ceramic Capacitor X7R 0603 (1608 Metric)"
 			(at 180.975 71.755 0)
 			(effects
@@
 			)
 		)
-		(property "MPN" ""
+		(property "MPN" "GMC10X7R104K50NT"
 			(at 180.975 71.755 0)
 			(effects
@@
 			)
 		)
-		(property "Digikey" ""
+		(property "Digikey" "https://www.digikey.de/en/products/detail/cal-chip-electronics-inc/GMC10X7R104K50NT/18151094"
 			(at 180.975 71.755 0)
 			(effects
@@
 			)
 		)
-		(property "Datasheet" "~"
+		(property "Datasheet" "https://calchip.com/wp-content/uploads/2023/09/GMC-Series-2.pdf"
 			(at 111.76 71.755 0)
 			(effects
@@
 			)
 		)
-		(property "Description" "Unpolarized capacitor, small symbol"
+		(property "Description" "0.1 µF ±10% 50V Ceramic Capacitor X7R 0603 (1608 Metric)"
 			(at 111.76 71.755 0)
 			(effects
@@
 			)
 		)
-		(property "MPN" ""
+		(property "MPN" "GMC10X7R104K50NT"
 			(at 111.76 71.755 0)
 			(effects
@@
 			)
 		)
-		(property "Digikey" ""
+		(property "Digikey" "https://www.digikey.de/en/products/detail/cal-chip-electronics-inc/GMC10X7R104K50NT/18151094"
 			(at 111.76 71.755 0)
 			(effects
